File: Hardware/Amplifier+Mixer.sch (EAGLE design)
At the start: 182 parts, among them IC1 7812, IC2 7805, IC3 7912, IC4 OPA134PA, IC5 OPA134PA, IC6 MEGA8-AI, IC7 74HCT04, J1 +12AC, J10 FAN, J2 0V, J3 -12AC, J4 PE, J5 TERMINAL-BLOCK-2PLUG-IN, J6 TERMINAL-BLOCK-2PLUG-IN, J7 ENCODER, J8 DISPLAY, J9 USB, K1 RELAY-F40.52, K2 RELAY-F40.52, Q1 NPN, U1 LM1117-3.3, U2 10k, U3 10k, U4 10k, U5 10k, U6 TDA7498L, U7 10k, U8 10k, X1 RCA-4-CHANNEL, X2 JST-XH2, X3 ICSP

Commit message: consolidated some components to minimize BOM
Parts:
- removed Q1: NPN, transistor-npn:BC817-16LT1SMD
- added R2, R52: 4k7, rcl:R-EU_R0603
- added T4: BC817, transistor:BC817-16-NPN-SOT23-BEC
- C66: value 104 -> 100n
- C67: value 105 -> 1µ
- D1, D3, D5, D7: value (none) -> 4007; device SparkFun-DiscreteSemi:DIODEBAS16 -> Parts:DIODE; MOUSER (none) -> 583-FM4007W-W; SPEC (none) -> 4007
- D10, D4, D8: value (none) -> 1N4148
- D2, D6: value DIODE -> 4007; MOUSER (none) -> 583-FM4007W-W; SPEC (none) -> 4007
- D9: value (none) -> 1N4148; device diode:DIODE-SOD123 -> SparkFun-DiscreteSemi:DIODEBAS16
- J1: value +12AC -> 6MM
- J10: value FAN -> JST-XH2
- J2: value 0V -> 6MM
- J3: value -12AC -> 6MM
- J4: value PE -> 6MM
- JP2: value bypass AC couple right -> (none)
- JP3: value bypass AC couple left -> (none)
- K1, K2: value RELAY-F40.52 -> 12V 8A; CONRAD (none) -> 629528 - 62; SPEC (none) -> Hongfa HF115F/012-2ZS4A
- R3: device rcl:R-EU_R1206 -> rcl:R-EU_R0603
- T1, T2, T3: value (none) -> BC817
Connections:
- net +3V3: now also R2.2, R52.2
- net AUDIO_DETECT: now also T4.C; no longer Q1.C
- net DGND: now also T4.E; no longer Q1.E
- net N$37: now also T4.B; no longer Q1.B
- net SCL: now also R52.1
- net SDA: now also R2.1
Other:
- note added: "3.3V and 5V digital Supply"
- note added: "Amplifier"
- note added: "Amplifier Power"
- note added: "DC COUPLE L"
- note added: "DC COUPLE R"
- note added: "Digital Pots"
- note added: "Display Connector & Level Shifting"
- note added: "Dual-Rail Power for Audio"
- note added: "Equalizer"
- note added: "Fan Controller"
- note added: "I2C-Pullups"
- note added: "Input Mixer"
- note added: "Input Signal Detection"
- note added: "Main Volume"
- note added: "Mechanical & Mounting"
- note added: "Power Button"
- note added: "Speaker Protect"
- note added: "Star-Ground Point"
- note added: "USB Power Out"
- note added: "µC & I/O"
- moved on the sheet: B1, C1, C10, C11, C12, C13, C14, C15, C16, C17, C18, C19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

Commit message: added order numbers for conrad and mouser as attributes of the parts
Parts:
- B1: MOUSER (none) -> 833-GBJL2510-BP; STOCK (none) -> 0
- C1, C13: value 220µ -> 220µ 25V; CONRAD (none) -> 404629 - 62; MOUSER (none) -> 647-UWT1E221MNL1GS; STOCK (none) -> 2
- C10, C14, C15, C18, C2, C21, C23, C24, C28, C29, C3, C34, C43, C49, C5, C52, C58, C62, C63, C64, C65, C66, C7, C8: CONRAD (none) -> 457901 - 62; MOUSER (none) -> 710-885012206071; STOCK (none) -> 24
- C11, C12: MOUSER (none) -> 647-LLS1H103MELC; STOCK (none) -> 0
- C16, C4: value 470µ -> 470µ 16V; CONRAD (none) -> 404626 - 62; MOUSER (none) -> 647-UWT1C471MNL1S; STOCK (none) -> 2
- C17, C27, C33, C39, C41, C48: MOUSER (none) -> 80-R82EC1100AA50K; STOCK (none) -> 0
- C19, C51: MOUSER (none) -> 594-222237188472; STOCK (none) -> 0
- C20, C22, C32, C37, C40, C57: MOUSER (none) -> 80-R82DC4100AA60K; STOCK (none) -> 0
- C25, C59: MOUSER (none) -> 505-FKP2J006801D00KS; STOCK (none) -> 0
- C26, C30, C31, C36, C42, C45, C46, C50: MOUSER (none) -> 80-R82DC3220AA60K; STOCK (none) -> 0
- C35, C44: MOUSER (none) -> 505-MKS2D034701E00JI; STOCK (none) -> 0
- C38, C47: MOUSER (none) -> 505-FKP2C003301D00KI; STOCK (none) -> 0
- C53, C54: CONRAD 458140 - 62 -> 1279028 - 62; MOUSER (none) -> 80-C1206C105M5RECLR; STOCK (none) -> 0
- C55, C56: MOUSER (none) -> 77-VJ1206Y104KXBAT; STOCK (none) -> 0
- C6, C9: value 4.7µ -> 4.7µ 10V; CONRAD (none) -> 1280266 - 62; MOUSER (none) -> 710-865230642008; STOCK (none) -> 2
- C60, C61: CONRAD (none) -> 421520 - 6; MOUSER (none) -> 710-865080642006; STOCK (none) -> 0
- C67: CONRAD (none) -> 457913 - 62; MOUSER (none) -> 710-885012106022; STOCK (none) -> 1
- D1, D2, D3, D5, D6, D7: CONRAD (none) -> 160493 - 62; STOCK (none) -> 6
- D10, D4, D8, D9: CONRAD (none) -> 1582023 - 62; MOUSER (none) -> 512-1N4148WS; STOCK (none) -> 4
- H1, H2, H3, H4: STOCK (none) -> 4
- IC1: CONRAD (none) -> 179230 - 62; MOUSER (none) -> 511-L7812CV; STOCK (none) -> 1
- IC2: CONRAD (none) -> 179205 - 62; MOUSER (none) -> 511-L7805CV; STOCK (none) -> 1
- IC3: CONRAD (none) -> 156077 - 62; MOUSER (none) -> 511-L7912CV; STOCK (none) -> 1
- IC4, IC5: MOUSER (none) -> 595-OPA134PA; STOCK (none) -> 0
- IC6: CONRAD (none) -> 155196 - 62; MOUSER (none) -> 556-ATMEGA328-AU; STOCK (none) -> 1
- IC7: CONRAD (none) -> 144614 - 62; MOUSER (none) -> 771-74HCT04D; STOCK (none) -> 1
- IC8, IC9: value (none) -> LM358D; CONRAD (none) -> 1010764 - 62; MOUSER (none) -> 511-LM358DT; STOCK (none) -> 2
- J1, J2, J3, J4: CONRAD (none) -> 808428 - 62; MOUSER (none) -> 571-726386-2; STOCK (none) -> 2
- J10, X2: CONRAD (none) -> 741161 - 62; MOUSER (none) -> 575-3191010200006000; STOCK (none) -> 2
- J5, J6: CONRAD (none) -> 1327203 - 62; MOUSER (none) -> 651-1954919; STOCK (none) -> 2
- J7, J8: CONRAD (none) -> 741206 - 62; MOUSER (none) -> 538-35312-0260; STOCK (none) -> 1
- J9: CONRAD (none) -> 1311468 - 62; MOUSER (none) -> 523-GSB19110KEU; STOCK (none) -> 0
- JP1, U$1: STOCK (none) -> 1
- JP2, JP3: CONRAD (none) -> 1560728 - 62; MOUSER (none) -> 200-TSW10223TS; STOCK (none) -> 2
- JP4: CONRAD (none) -> 1560647 - 62; MOUSER (none) -> 649-68001-204HLF; STOCK (none) -> 0
- JP5: CONRAD (none) -> 1390113 - 62; MOUSER (none) -> 710-61300611121; STOCK (none) -> 0
- K1, K2: MOUSER (none) -> 655-RT424012; STOCK (none) -> 0
- KK1, KK4: CONRAD (none) -> 188093 - 62; MOUSER (none) -> 490-HSE-B20254-035H; STOCK (none) -> 2
- KK2: CONRAD (none) -> 188158 - 62; MOUSER (none) -> 490-HSE-B2111-038; STOCK (none) -> 1
- L1, L2, L3, L4: value 22µ 2.8A -> 22µ 2.2A; MOUSER (none) -> 710-744771220; STOCK (none) -> 0
- R1: MOUSER (none) -> 279-EP5WS470RJ; STOCK (none) -> 0
- R10, R29, R30, R32, R33, R6, R7, R9: MOUSER (none) -> 71-SMM02070C5601FBP0; STOCK (none) -> 0
- R11, R14, R15, R18, R19, R21, R25, R26, R28, R35, R37, R38, R4, R40, R42, R5: MOUSER (none) -> 71-SMM02070C7501FBP0; STOCK (none) -> 0
- R12, R17, R31, R36, R39, R8: MOUSER (none) -> 756-WRM024HPC100KFT3; STOCK (none) -> 0
- R13, R3, R43, R44, R47: CONRAD (none) -> 1585269 - 62; MOUSER (none) -> 603-RC0603FR-0710KL; STOCK (none) -> 5
- R16, R22, R24, R34: MOUSER (none) -> 756-WRM0204HPC8R2FT3; STOCK (none) -> 0
- R2, R52: CONRAD (none) -> 1585263 - 62; MOUSER (none) -> 603-AC0603JR-134K7L; STOCK (none) -> 2
- R20, R23: MOUSER (none) -> 756-WRM0207HPC22RFT2; STOCK (none) -> 0
- R27: CONRAD (none) -> 1585778 - 62; MOUSER (none) -> 603-RC0603FR-0722RL; STOCK (none) -> 0
- R41: CONRAD (none) -> 1584631 - 62; MOUSER (none) -> 603-RC0603FR-0739KL; STOCK (none) -> 1
- R45, R50, R51: CONRAD (none) -> 1585255 - 62; MOUSER (none) -> 603-RC0603FR-071KL; STOCK (none) -> 3
- R46, R48, R49: CONRAD (none) -> 1585286 - 62; MOUSER (none) -> 71-RCA0603100KJNEC; STOCK (none) -> 3
- T1, T2, T3, T4: MOUSER (none) -> 863-BC817-16LT3G; STOCK (none) -> 6
- U1: CONRAD (none) -> 1261149 - 62; MOUSER (none) -> 926-LM1117MPX3.3NOPB; STOCK (none) -> 1
- U2, U3, U4, U5, U7, U8: CONRAD (none) -> 1083246 - 62; MOUSER (none) -> 579-MCP4641-103E/ST; STOCK (none) -> 6
- U6: MOUSER (none) -> 511-TDA7498TR; STOCK (none) -> 0
- VR1: value 10k -> 100k; CONRAD (none) -> 1618568 - 62; MOUSER (none) -> 858-35WR100KLFTR; STOCK (none) -> 0
- X1: CONRAD (none) -> 1578879 - 62; MOUSER (none) -> 806-KLP42X-61-WWRR; STOCK (none) -> 1
- X3: CONRAD (none) -> 1560967 - 62; MOUSER (none) -> 200-TSW10307TD; STOCK (none) -> 1
Connections:
- removed net N$46: U7R1.A, X1B.T2
- removed net N$47: U8R1.A, X1A.T2
- removed net N$48: U8R2.A, X1A.T1
- removed net N$49: U7R2.A, X1B.T1
- net AGND: now also U7R1.A, U7R2.A; no longer U7R1.B, U7R2.B, U8R1.B, U8R2.B
- net N$40: now also U7R2.B, X1B.T2; no longer R11.1, U8R1.W
- net N$41: now also U7R1.B, X1B.T1; no longer R19.1, U8R2.W
- net N$42: now also U7R1.W; no longer U7R2.W
- net N$43: now also U7R2.W; no longer U7R1.W
Other:
- note added: "Input: 160VA Load: 8 Ohms Imax = sqrt(160W / 8Ohm) = 4.5A Vripple =(Imax * (1 * 100Hz)) / 20mF = 2,25V"
- moved on the sheet: C15, C16, C3, C4, KK2, U7R1, U7R2, U8R1, U8R2

Commit message: first routing pass
Parts:
- added JP6: PREAMP OUT, pinhead:PINHD-2X3
- added R54, R55: 39k, rcl:R-EU_R0603
- added S1: GAIN SELECT, switch-dil:DIP02YL
- C20: value 1µ -> DC COUPLE L
- JP2: value (none) -> DC COULE R
- JP3: value (none) -> DC COUPLE L
- JP5: value EXPANSION -> MIX OUT; device pinhead:PINHD-1X6 -> pinhead:PINHD-2X3; CONRAD 1390113 - 62 -> (none); MOUSER 710-61300611121 -> (none); STOCK 0 -> (none)
Connections:
- net N$57 renamed INNB
- net N$58 renamed INPB
- net N$59 renamed INNA
- net N$60 renamed INPA
- removed net N$88: IC6.PC1(ADC1), JP5.5
- removed net N$89: IC6.PC2(ADC2), JP5.4
- removed net N$90: IC6.PC3(ADC3), JP5.3
- removed net N$91: K1SW1.O, R1.2
- new net AMP_MUTE_CL: R54.1, U6.MUTE
- new net AMP_STBY_CL: R55.1, U6.STBY
- new net EQ_L: IC4B.+IN, JP5.6
- new net EQ_R: IC4A.+IN, JP5.2
- new net N$46: U8R2.B, X1A.T2
- new net N$47: U8R1.B, X1A.T1
- new net N$48: R19.1, U8R1.W
- new net N$49: R11.1, U8R2.W
- new net N$57: S1.3, U6.GAIN1
- new net N$58: S1.4, U6.GAIN0
- new net N$59: K1SW2.O, R1.2
- new net N$81: C22.1, JP6.1
- new net N$84: C37.1, JP6.5
- net +18V: now also K1SW1.P; no longer K1SW2.P
- net +3V3: now also S1.1, S1.2; no longer JP5.6, U6.GAIN0, U6.GAIN1
- net -18V: now also K1SW2.P; no longer K1SW1.P
- net AGND: now also JP5.3, JP5.4, JP6.3, JP6.4, U2R1.A, U2R2.A, U8R1.A, U8R2.A; no longer U2R1.B, U2R2.B
- net AMP_MUTE: now also R54.2; no longer U6.MUTE
- net AMP_STBY: now also R55.2; no longer U6.STBY
- net DGND: no longer JP5.1, JP5.2, T1.E
- net EQ_OUT_L: now also U2R1.B; no longer U2R2.A
- net EQ_OUT_R: now also U2R2.B; no longer U2R1.A
- net GND: now also T1.E
- net L_OUT-: now also J6G$1.P$1; no longer J6G$2.P$1
- net MIX_L: now also JP5.5; no longer IC4B.+IN
- net MIX_R: now also JP5.1; no longer IC4A.+IN
- net N$27: now also K1SW2.S; no longer K1SW1.S
- net N$51: now also J6G$2.P$1; no longer J6G$1.P$1
- net N$53: now also K1SW1.O; no longer K1SW2.S
- net N$9: now also K1SW1.S; no longer K1SW2.O
- net PREAMP_OUT_L: now also JP6.6, U2R1.W; no longer C37.1, U2R2.W
- net PREAMP_OUT_R: now also JP6.2, U2R2.W; no longer C22.1, U2R1.W
- net SCL: now also IC7A.I; no longer IC7B.I
- net SCL_5V: now also IC7F.O; no longer IC7E.O
- net SDA: now also IC7B.I; no longer IC7A.I
- net SDA_5V: now also IC7E.O; no longer IC7F.O
Other:
- note added: "AC coupling cut-off: 1/(2πCR) R = 60k (from Datasheet) fcut = 1/(2π1µ60k) = 2,6Hz"
- moved on the sheet: IC7A, IC7B, IC7E, IC7F, JP5, K1, U2R1, U2R2

Commit message: first silkscreen placement pass
Parts:
- added JP10: PEGND, SparkFun-Jumpers:JUMPER-SMT_2_NO_NO-SILK
- added JP7, JP8, JP9: (no value), pinhead:PINHD-1X2
Connections:
- net N$57 renamed GAIN1
- net N$58 renamed GAIN0
- net +12V: now also JP7.2
- net +3V3: now also JP9.2
- net -12V: now also JP8.2
- net DGND: now also JP9.1
- net GND: now also JP10.1, JP7.1, JP8.1
- net PE: now also JP10.2
Other:
- moved on the sheet: C1, C10, C13, C14, C15, C16, C2, C3, C4, C5, C6, C7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

Commit message: added temp sensor for amp chip heatsink
Parts:
- added U9: MCP9700SMD, SparkFun-Sensors:MCP9700SMD
- renumbered U$1 to KK3
Connections:
- new net T_SENSE: IC6.PC1(ADC1), U9.VO
- net +3V3: now also U9.VCC
- net DGND: now also U9.GND
Changed lines of the file:
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@@
 <part name="SUPPLY37" library="supply2" library_urn="urn:adsk.eagle:library:372" deviceset="DGND" device=""/>
 <part name="PE3" library="supply1" library_urn="urn:adsk.eagle:library:371" deviceset="PE" device=""/>
-<part name="U$1" library="Class D Amp" library_urn="urn:adsk.eagle:library:8719353" deviceset="HEATSINK-PENTIUM" device="" package3d_urn="urn:adsk.eagle:package:8803895/4">
+<part name="KK3" library="Class D Amp" library_urn="urn:adsk.eagle:library:8719353" deviceset="HEATSINK-PENTIUM" device="" package3d_urn="urn:adsk.eagle:package:8803895/4">
 <attribute name="STOCK" value="1"/>
 </part>
@@
 <part name="JP10" library="SparkFun-Jumpers" library_urn="urn:adsk.eagle:library:528" deviceset="JUMPER-SMT_2_NO" device="_NO-SILK" package3d_urn="urn:adsk.eagle:package:39277/1" value="PEGND"/>
 <part name="PE4" library="supply1" library_urn="urn:adsk.eagle:library:371" deviceset="PE" device=""/>
+<part name="U9" library="SparkFun-Sensors" deviceset="MCP9700" device="SMD"/>
+<part name="+3V2" library="supply1" library_urn="urn:adsk.eagle:library:371" deviceset="+3V3" device=""/>
+<part name="SUPPLY5" library="supply2" library_urn="urn:adsk.eagle:library:372" deviceset="DGND" device=""/>
 </parts>
 <sheets>
@@
 <text x="236.22" y="101.6" size="1.778" layer="97" align="bottom-center">EQ Base</text>
 <text x="236.22" y="124.46" size="1.778" layer="97" align="bottom-center">Master Volume</text>
-<wire x1="487.68" y1="152.4" x2="487.68" y2="223.52" width="0.1524" layer="97" style="longdash"/>
-<wire x1="487.68" y1="223.52" x2="657.86" y2="223.52" width="0.1524" layer="97" style="longdash"/>
+<wire x1="502.92" y1="152.4" x2="502.92" y2="223.52" width="0.1524" layer="97" style="longdash"/>
+<wire x1="502.92" y1="223.52" x2="657.86" y2="223.52" width="0.1524" layer="97" style="longdash"/>
 <wire x1="657.86" y1="223.52" x2="657.86" y2="152.4" width="0.1524" layer="97" style="longdash"/>
-<wire x1="657.86" y1="152.4" x2="487.68" y2="152.4" width="0.1524" layer="97" style="longdash"/>
+<wire x1="657.86" y1="152.4" x2="502.92" y2="152.4" width="0.1524" layer="97" style="longdash"/>
 <wire x1="325.12" y1="0" x2="325.12" y2="149.86" width="0.1524" layer="97" style="longdash"/>
 <wire x1="325.12" y1="149.86" x2="459.74" y2="149.86" width="0.1524" layer="97" style="longdash"/>
@@
 R = 60k (from Datasheet)
 fcut = 1/(2π1µ60k) = 2,6Hz</text>
+<wire x1="462.28" y1="152.4" x2="462.28" y2="223.52" width="0.1524" layer="97" style="longdash"/>
+<wire x1="462.28" y1="223.52" x2="500.38" y2="223.52" width="0.1524" layer="97" style="longdash"/>
+<wire x1="500.38" y1="223.52" x2="500.38" y2="152.4" width="0.1524" layer="97" style="longdash"/>
+<wire x1="500.38" y1="152.4" x2="462.28" y2="152.4" width="0.1524" layer="97" style="longdash"/>
 </plain>
 <instances>
@@
 <attribute name="VALUE" x="342.9" y="186.182" size="1.778" layer="96" align="top-center"/>
 </instance>
-<instance part="U$1" gate="G$1" x="551.18" y="104.14" smashed="yes">
+<instance part="KK3" gate="G$1" x="551.18" y="104.14" smashed="yes">
 <attribute name="NAME" x="556.895" y="107.315" size="1.778" layer="95"/>
 <attribute name="VALUE" x="556.895" y="104.775" size="1.778" layer="96"/>
@@
 <attribute name="VALUE" x="424.18" y="158.242" size="1.778" layer="96" align="top-center"/>
 </instance>
+<instance part="U9" gate="G$1" x="474.98" y="185.42" smashed="yes">
+<attribute name="NAME" x="467.36" y="191.008" size="1.778" layer="95"/>
+<attribute name="VALUE" x="477.52" y="191.008" size="1.778" layer="96"/>
+</instance>
+<instance part="+3V2" gate="G$1" x="464.82" y="198.12" smashed="yes">
+<attribute name="VALUE" x="464.82" y="198.374" size="1.778" layer="96" align="bottom-center"/>
+</instance>
+<instance part="SUPPLY5" gate="G$1" x="474.98" y="175.26" smashed="yes">
+<attribute name="VALUE" x="474.98" y="173.736" size="1.778" layer="96" align="top-center"/>
+</instance>
 </instances>
 <busses>
@@
 <junction x="513.08" y="25.4"/>
 </segment>
+<segment>
+<pinref part="U9" gate="G$1" pin="VCC"/>
+<pinref part="+3V2" gate="G$1" pin="+3V3"/>
+<wire x1="464.82" y1="187.96" x2="464.82" y2="195.58" width="0.1524" layer="91"/>
+</segment>
 </net>
 <net name="N$37" class="0">
@@
 <wire x1="363.22" y1="190.5" x2="363.22" y2="187.96" width="0.1524" layer="91"/>
 </segment>
+<segment>
+<pinref part="U9" gate="G$1" pin="GND"/>
+<pinref part="SUPPLY5" gate="G$1" pin="DGND"/>
+<wire x1="474.98" y1="180.34" x2="474.98" y2="177.8" width="0.1524" layer="91"/>
+</segment>
 </net>
 <net name="AGND" class="0">
@@
 </segment>
 </net>
+<net name="T_SENSE" class="0">
+<segment>
+<pinref part="U9" gate="G$1" pin="VO"/>
+<wire x1="485.14" y1="187.96" x2="487.68" y2="187.96" width="0.1524" layer="91"/>
+<label x="487.68" y="187.96" size="1.27" layer="95" xref="yes"/>
+</segment>
+<segment>
+<pinref part="IC6" gate="G$1" pin="PC1(ADC1)"/>
+<wire x1="81.28" y1="99.06" x2="83.82" y2="99.06" width="0.1524" layer="91" style="longdash"/>
+<label x="83.82" y="99.06" size="1.27" layer="95" xref="yes"/>
+</segment>
+</net>

Commit message: added power led connector
Parts:
- added D11, D12: 1N4148, SparkFun-DiscreteSemi:DIODEBAS16
- added X4: JST-XH2, Class D Amp:JST-XH2
Connections:
- new net N$57: C8.1, D11.C, D12.C, U1.IN
- new net POWER_LED: IC6.PC2(ADC2), X4.2
- new net VPP: D12.A, X32.S
- net +12V: now also D11.A; no longer C8.1, U1.IN
- net +3V3: no longer X32.S
- net DGND: now also X4.1
Other:
- moved on the sheet: X2

Commit message: removed 74hct04 for level shifting
Parts:
- removed IC7: 74HCT04, 74xx-eu:7404D
- removed R43: 10k, rcl:R-EU_R0603
- removed T4: BC817, transistor:BC817-16-NPN-SOT23-BEC
Connections:
- removed net N$37: R45.1, T4.B
- removed net N$60: IC7A.O, IC7F.I
- removed net N$83: IC7B.O, IC7E.I
- removed net SCL_5V: IC7F.O, J8.4
- removed net SDA_5V: IC7E.O, J8.3
- net +3V3: no longer R43.1
- net +5V: no longer IC7C.I, IC7D.I, IC7P.VCC
- net AUDIO_DETECT: now also R45.1; no longer R43.2, T4.C
- net DGND: no longer IC7P.GND, T4.E
- net SCL: now also J8.4; no longer IC7A.I
- net SDA: now also J8.3; no longer IC7B.I
Other:
- note added: "Display Connector"
- note removed: "Display Connector & Level Shifting"
