File: Hardware/Amplifier+Mixer.sch (EAGLE design)
At the start: 193 parts, among them IC1 7812, IC2 7805, IC3 7912, IC4 OPA134PA, IC5 OPA134PA, IC6 MEGA8-AI, IC8 LM358D, IC9 LM358D, J1 6MM, J10 JST-XH2, J2 6MM, J3 6MM, J4 6MM, J5 TERMINAL-BLOCK-2PLUG-IN, J6 TERMINAL-BLOCK-2PLUG-IN, J7 ENCODER, J8 DISPLAY, J9 USB, K1 12V 8A, K2 12V 8A, T1 BC817, T2 BC817, T3 BC817, U1 LM1117-3.3, U2 10k, U3 10k, U4 10k, U5 10k, U6 TDA7498L, U7 10k, U8 10k, U9 MCP9700SMD, X1 RCA-4-CHANNEL, X2 JST-XH2, X3 ICSP, X4 JST-XH2

Commit message: removed gain selection dip switch and wired gain pins to µC
Parts:
- removed S1: GAIN SELECT, switch-dil:DIP02YL
Connections:
- removed net N$79: IC6.PB4(MISO), X31.S
- removed net N$80: IC6.PB5(SCK), X33.S
- net +3V3: no longer S1.1, S1.2
- net GAIN0: now also IC6.PB4(MISO), X31.S; no longer S1.4
- net GAIN1: now also IC6.PB5(SCK), X33.S; no longer S1.3
Other:
- moved on the sheet: X31, X32, X33, X36
Changed lines of the file:
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@@
 <part name="PE2" library="supply1" library_urn="urn:adsk.eagle:library:371" deviceset="PE" device=""/>
 <part name="+3V312" library="supply1" library_urn="urn:adsk.eagle:library:371" deviceset="+3V3" device=""/>
-<part name="+3V317" library="supply1" library_urn="urn:adsk.eagle:library:371" deviceset="+3V3" device=""/>
 <part name="C49" library="rcl" library_urn="urn:adsk.eagle:library:334" deviceset="C-EU" device="C0603" package3d_urn="urn:adsk.eagle:package:23616/2" value="100n">
 <spice>
@@
 <attribute name="STOCK" value="3"/>
 </part>
-<part name="S1" library="switch-dil" library_urn="urn:adsk.eagle:library:375" deviceset="DIP02YL" device="" package3d_urn="urn:adsk.eagle:package:27254/2" value="GAIN SELECT"/>
 <part name="GND5" library="supply1" library_urn="urn:adsk.eagle:library:371" deviceset="GND" device=""/>
 <part name="JP5" library="pinhead" library_urn="urn:adsk.eagle:library:325" deviceset="PINHD-2X3" device="" package3d_urn="urn:adsk.eagle:package:22462/2" value="MIX OUT"/>
@@
 <attribute name="VALUE" x="502.92" y="71.374" size="1.778" layer="96" align="bottom-center"/>
 </instance>
-<instance part="+3V317" gate="G$1" x="513.08" y="27.94" smashed="yes">
-<attribute name="VALUE" x="513.08" y="28.194" size="1.778" layer="96" align="bottom-center"/>
-</instance>
 <instance part="C49" gate="G$1" x="525.78" y="53.34" smashed="yes">
 <attribute name="NAME" x="523.748" y="50.5968" size="1.778" layer="95" rot="R180" align="top-left"/>
@@
 <attribute name="STOCK" x="27.94" y="109.22" size="1.778" layer="96" display="off"/>
 </instance>
-<instance part="SUPPLY21" gate="G$1" x="91.44" y="27.94" smashed="yes">
-<attribute name="VALUE" x="91.44" y="26.416" size="1.778" layer="96" align="top-center"/>
+<instance part="SUPPLY21" gate="G$1" x="91.44" y="17.78" smashed="yes">
+<attribute name="VALUE" x="91.44" y="16.256" size="1.778" layer="96" align="top-center"/>
 </instance>
 <instance part="P+10" gate="1" x="685.8" y="48.26" smashed="yes">
@@
 <attribute name="PART" x="673.1" y="68.58" size="1.778" layer="95"/>
 </instance>
-<instance part="X3" gate="1" x="101.6" y="45.72" smashed="yes">
-<attribute name="NAME" x="102.616" y="44.958" size="1.524" layer="95"/>
-<attribute name="CONRAD" x="101.6" y="45.72" size="1.778" layer="96" display="off"/>
-<attribute name="MOUSER" x="101.6" y="45.72" size="1.778" layer="96" display="off"/>
-<attribute name="STOCK" x="101.6" y="45.72" size="1.778" layer="96" display="off"/>
+<instance part="X3" gate="1" x="101.6" y="43.18" smashed="yes">
+<attribute name="NAME" x="102.616" y="42.418" size="1.524" layer="95"/>
+<attribute name="CONRAD" x="101.6" y="43.18" size="1.778" layer="96" display="off"/>
+<attribute name="MOUSER" x="101.6" y="43.18" size="1.778" layer="96" display="off"/>
+<attribute name="STOCK" x="101.6" y="43.18" size="1.778" layer="96" display="off"/>
 </instance>
-<instance part="X3" gate="2" x="101.6" y="35.56" smashed="yes">
-<attribute name="NAME" x="102.616" y="34.798" size="1.524" layer="95"/>
+<instance part="X3" gate="2" x="101.6" y="25.4" smashed="yes">
+<attribute name="NAME" x="102.616" y="24.638" size="1.524" layer="95"/>
 </instance>
-<instance part="X3" gate="3" x="101.6" y="43.18" smashed="yes">
-<attribute name="NAME" x="102.616" y="42.418" size="1.524" layer="95"/>
+<instance part="X3" gate="3" x="101.6" y="38.1" smashed="yes">
+<attribute name="NAME" x="102.616" y="37.338" size="1.524" layer="95"/>
 </instance>
 <instance part="X3" gate="4" x="101.6" y="48.26" smashed="yes">
@@
 <attribute name="NAME" x="21.082" y="120.396" size="1.524" layer="95" rot="R90"/>
 </instance>
-<instance part="X3" gate="6" x="101.6" y="33.02" smashed="yes">
-<attribute name="NAME" x="102.616" y="32.258" size="1.524" layer="95"/>
+<instance part="X3" gate="6" x="101.6" y="22.86" smashed="yes">
+<attribute name="NAME" x="102.616" y="22.098" size="1.524" layer="95"/>
 </instance>
 <instance part="X2" gate="G$1" x="375.92" y="190.5" smashed="yes" rot="MR0">
@@
 <attribute name="STOCK" x="525.78" y="15.24" size="1.778" layer="96" display="off"/>
 </instance>
-<instance part="S1" gate="1" x="523.24" y="25.4" smashed="yes" rot="R270">
-<attribute name="NAME" x="518.16" y="27.94" size="1.778" layer="95"/>
-<attribute name="VALUE" x="518.16" y="18.415" size="1.778" layer="96"/>
-</instance>
 <instance part="GND5" gate="1" x="149.86" y="170.18" smashed="yes">
 <attribute name="VALUE" x="147.32" y="167.64" size="1.778" layer="96"/>
@@
 <attribute name="VALUE" x="474.98" y="173.736" size="1.778" layer="96" align="top-center"/>
 </instance>
-<instance part="SUPPLY36" gate="G$1" x="91.44" y="40.64" smashed="yes">
-<attribute name="VALUE" x="89.535" y="43.815" size="1.778" layer="96"/>
+<instance part="SUPPLY36" gate="G$1" x="91.44" y="30.48" smashed="yes">
+<attribute name="VALUE" x="89.535" y="33.655" size="1.778" layer="96"/>
 </instance>
 <instance part="D11" gate="G$1" x="264.16" y="195.58" smashed="yes" rot="R270">
@@
 </segment>
 <segment>
-<pinref part="+3V317" gate="G$1" pin="+3V3"/>
-<pinref part="S1" gate="1" pin="1"/>
-<wire x1="513.08" y1="25.4" x2="515.62" y2="25.4" width="0.1524" layer="91"/>
-<pinref part="S1" gate="1" pin="2"/>
-<wire x1="515.62" y1="22.86" x2="513.08" y2="22.86" width="0.1524" layer="91"/>
-<wire x1="513.08" y1="22.86" x2="513.08" y2="25.4" width="0.1524" layer="91"/>
-<junction x="513.08" y="25.4"/>
-</segment>
-<segment>
 <pinref part="U9" gate="G$1" pin="VCC"/>
 <pinref part="+3V2" gate="G$1" pin="+3V3"/>
@@
 </segment>
 <segment>
-<wire x1="96.52" y1="33.02" x2="91.44" y2="33.02" width="0.1524" layer="91"/>
+<wire x1="96.52" y1="22.86" x2="91.44" y2="22.86" width="0.1524" layer="91"/>
 <pinref part="SUPPLY21" gate="G$1" pin="DGND"/>
-<wire x1="91.44" y1="33.02" x2="91.44" y2="30.48" width="0.1524" layer="91"/>
+<wire x1="91.44" y1="22.86" x2="91.44" y2="20.32" width="0.1524" layer="91"/>
 <pinref part="X3" gate="6" pin="S"/>
 </segment>
@@
 </segment>
 </net>
-<net name="N$79" class="0">
-<segment>
-<pinref part="IC6" gate="G$1" pin="PB4(MISO)"/>
-<wire x1="96.52" y1="45.72" x2="81.28" y2="45.72" width="0.1524" layer="91"/>
-<pinref part="X3" gate="1" pin="S"/>
-</segment>
-</net>
-<net name="N$80" class="0">
-<segment>
-<pinref part="IC6" gate="G$1" pin="PB5(SCK)"/>
-<wire x1="96.52" y1="43.18" x2="81.28" y2="43.18" width="0.1524" layer="91"/>
-<pinref part="X3" gate="3" pin="S"/>
-</segment>
-</net>
 <net name="N$82" class="0">
 <segment>
@@
 <segment>
 <pinref part="U6" gate="G$1" pin="GAIN1"/>
-<pinref part="S1" gate="1" pin="3"/>
-<wire x1="530.86" y1="22.86" x2="533.4" y2="22.86" width="0.1524" layer="91"/>
+<wire x1="518.16" y1="22.86" x2="533.4" y2="22.86" width="0.1524" layer="91"/>
+<label x="518.16" y="22.86" size="1.27" layer="95" rot="R180" xref="yes"/>
+</segment>
+<segment>
+<pinref part="IC6" gate="G$1" pin="PB5(SCK)"/>
+<wire x1="96.52" y1="38.1" x2="86.36" y2="38.1" width="0.1524" layer="91"/>
+<wire x1="86.36" y1="38.1" x2="86.36" y2="43.18" width="0.1524" layer="91"/>
+<wire x1="86.36" y1="43.18" x2="81.28" y2="43.18" width="0.1524" layer="91"/>
+<pinref part="X3" gate="3" pin="S"/>
+<label x="96.52" y="40.64" size="1.27" layer="95" xref="yes"/>
+<wire x1="96.52" y1="40.64" x2="96.52" y2="38.1" width="0.1524" layer="91"/>
+<junction x="96.52" y="38.1"/>
 </segment>
 </net>
@@
 <segment>
 <pinref part="U6" gate="G$1" pin="GAIN0"/>
-<pinref part="S1" gate="1" pin="4"/>
-<wire x1="530.86" y1="25.4" x2="533.4" y2="25.4" width="0.1524" layer="91"/>
+<wire x1="518.16" y1="25.4" x2="533.4" y2="25.4" width="0.1524" layer="91"/>
+<label x="518.16" y="25.4" size="1.27" layer="95" rot="R180" xref="yes"/>
+</segment>
+<segment>
+<pinref part="IC6" gate="G$1" pin="PB4(MISO)"/>
+<wire x1="96.52" y1="43.18" x2="88.9" y2="43.18" width="0.1524" layer="91"/>
+<wire x1="88.9" y1="43.18" x2="88.9" y2="45.72" width="0.1524" layer="91"/>
+<wire x1="88.9" y1="45.72" x2="81.28" y2="45.72" width="0.1524" layer="91"/>
+<pinref part="X3" gate="1" pin="S"/>
+<wire x1="96.52" y1="43.18" x2="96.52" y2="45.72" width="0.1524" layer="91"/>
+<junction x="96.52" y="43.18"/>
+<label x="96.52" y="45.72" size="1.27" layer="95" xref="yes"/>
 </segment>
 </net>
@@
 <segment>
 <pinref part="X3" gate="2" pin="S"/>
-<wire x1="96.52" y1="35.56" x2="91.44" y2="35.56" width="0.1524" layer="91" style="longdash"/>
+<wire x1="96.52" y1="25.4" x2="91.44" y2="25.4" width="0.1524" layer="91" style="longdash"/>
 <pinref part="SUPPLY36" gate="G$1" pin="VPP"/>
-<wire x1="91.44" y1="35.56" x2="91.44" y2="38.1" width="0.1524" layer="91" style="longdash"/>
+<wire x1="91.44" y1="25.4" x2="91.44" y2="27.94" width="0.1524" layer="91" style="longdash"/>
 </segment>
 <segment>
